Commit message: feat(botlab_diff_description): 更新机器人模型和启动配置

File: part3/ros2_ws/src/botlab_diff_description/urdf/diff_drive_car.urdf.xacro (robot description, xacro)
@@ -2,7 +2,7 @@
 <robot xmlns:xacro="http://www.ros.org/wiki/xacro" name="diff_drive_car">
   <!-- 参数定义 -->
-  <xacro:property name="chassis_length" value="0.5"/>     <!-- 底盘长度 50cm -->
-  <xacro:property name="chassis_width"  value="0.3"/>     <!-- 底盘宽度 30cm -->
-  <xacro:property name="chassis_height" value="0.08"/>    <!-- 底盘高度 8cm（略调低） -->
+  <xacro:property name="chassis_length" value="0.26"/>     <!-- 底盘长度 26cm -->
+  <xacro:property name="chassis_width"  value="0.22"/>     <!-- 底盘宽度 22cm -->
+  <xacro:property name="chassis_height" value="0.08"/>    <!-- 底盘高度 8cm -->
   <xacro:property name="wheel_radius"   value="0.0325"/>  <!-- 轮子半径 3.25cm（直径6.5cm） -->
   <xacro:property name="wheel_width"    value="0.02"/>    <!-- 轮胎厚度 2cm -->
@@ -15,5 +15,4 @@
         <box size="${chassis_length} ${chassis_width} ${chassis_height}"/>
       </geometry>
-      <!-- 底盘放在轮子上方 -->
       <origin xyz="0 0 ${wheel_radius + chassis_height/2}" rpy="0 0 0"/>
       <material name="blue">
@@ -31,4 +30,8 @@
       <inertia ixx="0.1" ixy="0" ixz="0" iyy="0.1" iyz="0" izz="0.1"/>
     </inertial>
+    <!-- Gazebo 物理标签 -->
+    <gazebo reference="base_link">
+      <material>Gazebo/Blue</material>
+    </gazebo>
   </link>
   <!-- 定义轮子模板 -->
@@ -54,4 +57,8 @@
         <inertia ixx="0.001" ixy="0" ixz="0" iyy="0.001" iyz="0" izz="0.001"/>
       </inertial>
+      <!-- Gazebo 物理属性 -->
+      <gazebo reference="wheel_${prefix}">
+        <material>Gazebo/Black</material>
+      </gazebo>
     </link>
     <joint name="joint_${prefix}" type="continuous">

Commit message: feat(urdf): 添加差速驱动插件并调整物理参数

File: part3/ros2_ws/src/botlab_diff_description/urdf/diff_drive_car.urdf.xacro (robot description, xacro)
@@ -1,4 +1,6 @@
 <?xml version="1.0"?>
 <robot xmlns:xacro="http://www.ros.org/wiki/xacro" name="diff_drive_car">
+  <!-- 引入差速驱动插件 -->
+  <xacro:include filename="$(find botlab_diff_description)/urdf/gazebo_control_plugin.xacro"/>
   <!-- 参数定义 -->
   <xacro:property name="chassis_length" value="0.26"/>     <!-- 底盘长度 26cm -->
@@ -27,6 +29,6 @@
     </collision>
     <inertial>
-      <mass value="5.0"/>
-      <inertia ixx="0.1" ixy="0" ixz="0" iyy="0.1" iyz="0" izz="0.1"/>
+      <mass value="2.0"/>
+      <inertia ixx="0.05" ixy="0" ixz="0" iyy="0.05" iyz="0" izz="0.08"/>
     </inertial>
     <!-- Gazebo 物理标签 -->
@@ -54,18 +56,25 @@
       </collision>
       <inertial>
-        <mass value="0.2"/>
-        <inertia ixx="0.001" ixy="0" ixz="0" iyy="0.001" iyz="0" izz="0.001"/>
+        <mass value="0.1"/>
+        <inertia ixx="0.0005" ixy="0" ixz="0" iyy="0.0005" iyz="0" izz="0.0005"/>
       </inertial>
       <!-- Gazebo 物理属性 -->
       <gazebo reference="wheel_${prefix}">
         <material>Gazebo/Black</material>
+        <mu1>1.0</mu1>
+        <mu2>1.0</mu2>
+        <kp>1000000.0</kp>
+        <kd>100.0</kd>
+        <minDepth>0.001</minDepth>
+        <maxVel>1.0</maxVel>
       </gazebo>
     </link>
     <joint name="joint_${prefix}" type="continuous">
-      <parent link="base_link"/>
-      <child link="wheel_${prefix}"/>
-      <origin xyz="${x} ${y} ${wheel_radius}" rpy="0 0 0"/>
-      <axis xyz="0 1 0"/>
-    </joint>
+        <parent link="base_link"/>
+        <child link="wheel_${prefix}"/>
+        <origin xyz="${x} ${y} ${wheel_radius}" rpy="0 0 0"/>
+        <axis xyz="0 1 0"/>
+        <dynamics damping="0.1" friction="0.1"/>
+      </joint>
   </xacro:macro>
   <!-- 四个轮子 -->
@@ -74,3 +83,5 @@
   <xacro:wheel prefix="rl" x="-${wheelbase/2}"  y="${ track/2}"/>
   <xacro:wheel prefix="rr" x="-${wheelbase/2}"  y="-${ track/2}"/>
+  <!-- 使用差速驱动插件 -->
+  <xacro:gazebo_control_plugin/>
 </robot>

Commit message: feat(gazebo_launch): 优化 Gazebo 启动方式并调整模型加载延迟

File: part3/ros2_ws/src/botlab_diff_description/urdf/diff_drive_car.urdf.xacro (robot description, xacro)
@@ -32,9 +32,9 @@
       <inertia ixx="0.05" ixy="0" ixz="0" iyy="0.05" iyz="0" izz="0.08"/>
     </inertial>
-    <!-- Gazebo 物理标签 -->
-    <gazebo reference="base_link">
-      <material>Gazebo/Blue</material>
-    </gazebo>
   </link>
+  <!-- Gazebo 物理标签 -->
+  <gazebo reference="base_link">
+    <material>Gazebo/Red</material>
+  </gazebo>
   <!-- 定义轮子模板 -->
   <xacro:macro name="wheel" params="prefix x y">
@@ -59,14 +59,4 @@
         <inertia ixx="0.0005" ixy="0" ixz="0" iyy="0.0005" iyz="0" izz="0.0005"/>
       </inertial>
-      <!-- Gazebo 物理属性 -->
-      <gazebo reference="wheel_${prefix}">
-        <material>Gazebo/Black</material>
-        <mu1>1.0</mu1>
-        <mu2>1.0</mu2>
-        <kp>1000000.0</kp>
-        <kd>100.0</kd>
-        <minDepth>0.001</minDepth>
-        <maxVel>1.0</maxVel>
-      </gazebo>
     </link>
     <joint name="joint_${prefix}" type="continuous">
@@ -78,4 +68,14 @@
       </joint>
   </xacro:macro>
+  <!-- Gazebo 物理属性 -->
+  <gazebo reference="wheel_${prefix}">
+    <material>Gazebo/Black</material>
+    <mu1>1.0</mu1>
+    <mu2>1.0</mu2>
+    <kp>1000000.0</kp>
+    <kd>100.0</kd>
+    <minDepth>0.001</minDepth>
+    <maxVel>1.0</maxVel>
+  </gazebo>
   <!-- 四个轮子 -->
   <xacro:wheel prefix="fl" x="${ wheelbase/2}"  y="${ track/2}"/>
