Commit message: refactor(botlab_zero): 更新机器人物理参数和控制器配置

File: part3/ros2_ws/src/botlab_diff_description/urdf/botlab_zero/base.urdf.xacro (robot description, xacro)
@@ -19,7 +19,7 @@
       </collision>
       <inertial>
-        <mass value="5.0"/>
-        <inertia ixx="0.1" ixy="0" ixz="0"
-                 iyy="0.1" iyz="0" izz="0.1"/>
+        <mass value="0.5"/>
+        <inertia ixx="0.01" ixy="0" ixz="0"
+                 iyy="0.01" iyz="0" izz="0.01"/>
       </inertial>
     </link>

File: part3/ros2_ws/src/botlab_diff_description/urdf/botlab_zero/botlab_zero.urdf.xacro (robot description, xacro)
@@ -40,32 +40,30 @@
                wheel_radius="${wheel_radius}"
                wheel_width="${wheel_width}"/>
-  <!-- ros2_control transmission -->
-  <xacro:diff_drive_control prefix="botlab_zero"/>
-<!-- ros2_control system -->
-<ros2_control name="botlab_zero_hw" type="system">
-  <hardware>
-    <plugin>gazebo_ros2_control/GazeboSystem</plugin>
-  </hardware>
-  <joint name="joint_fl">
-    <command_interface name="velocity"/>
-    <state_interface name="position"/>
-    <state_interface name="velocity"/>
-  </joint>
-  <joint name="joint_fr">
-    <command_interface name="velocity"/>
-    <state_interface name="position"/>
-    <state_interface name="velocity"/>
-  </joint>
-  <joint name="joint_rl">
-    <command_interface name="velocity"/>
-    <state_interface name="position"/>
-    <state_interface name="velocity"/>
-  </joint>
-  <joint name="joint_rr">
-    <command_interface name="velocity"/>
-    <state_interface name="position"/>
-    <state_interface name="velocity"/>
-  </joint>
-</ros2_control>
+  <!-- ros2_control system -->
+  <ros2_control name="botlab_zero_hw" type="system">
+    <hardware>
+      <plugin>gazebo_ros2_control/GazeboSystem</plugin>
+    </hardware>
+    <joint name="joint_fl">
+      <command_interface name="velocity"/>
+      <state_interface name="position"/>
+      <state_interface name="velocity"/>
+    </joint>
+    <joint name="joint_fr">
+      <command_interface name="velocity"/>
+      <state_interface name="position"/>
+      <state_interface name="velocity"/>
+    </joint>
+    <joint name="joint_rl">
+      <command_interface name="velocity"/>
+      <state_interface name="position"/>
+      <state_interface name="velocity"/>
+    </joint>
+    <joint name="joint_rr">
+      <command_interface name="velocity"/>
+      <state_interface name="position"/>
+      <state_interface name="velocity"/>
+    </joint>
+  </ros2_control>
   <!-- Gazebo 配置 -->
   <gazebo reference="base_link">
@@ -73,7 +71,13 @@
     <mu2>1.0</mu2>
     <material>Gazebo/Blue</material>
-    <!-- ROS2 Control 插件 -->
+  </gazebo>
+  <!-- ROS2 Control 插件 -->
+  <gazebo>
     <plugin name="gazebo_ros2_control" filename="libgazebo_ros2_control.so">
       <parameters>$(find botlab_diff_description)/config/botlab_zero_controllers.yaml</parameters>
+      <ros>
+        <remapping>/diff_drive_controller/cmd_vel_unstamped:=/cmd_vel</remapping>
+        <remapping>/diff_drive_controller/odom:=/odom</remapping>
+      </ros>
     </plugin>
   </gazebo>

File: part3/ros2_ws/src/botlab_diff_description/urdf/botlab_zero/wheel.urdf.xacro (robot description, xacro)
@@ -19,7 +19,7 @@
       </collision>
       <inertial>
-        <mass value="0.15"/>
-        <inertia ixx="0.001" ixy="0" ixz="0"
-                 iyy="0.001" iyz="0" izz="0.001"/>
+        <mass value="0.05"/>
+        <inertia ixx="0.0001" ixy="0" ixz="0"
+                 iyy="0.0001" iyz="0" izz="0.0001"/>
       </inertial>
     </link>
